File: Hardware/stm32f103.sch (KiCad schematic (older format))
At the start: 13 parts, among them U2 STM32F103C8Tx

Commit message: forgot to save
Connections:
- net Currrent_ADC: now reaches U2.11 (PA1)
- net ADC renamed Vin_ADC
- no-connect marks 26 -> 25
Changed lines of the file:
@@
 	6500 3100 6850 3100
 Text HLabel 6850 3100 2    50   Input ~ 0
-ADC
+Vin_ADC
 Wire Wire Line
 	5900 1800 6000 1800
@@
 NoConn ~ 6500 3400
 NoConn ~ 6500 3300
-NoConn ~ 6500 3200
 $Comp
 L power:VDDA #PWR0122
@@
 Wire Wire Line
 	5700 1700 5900 1700
+Wire Wire Line
+	6500 3200 6850 3200
+Text HLabel 6850 3200 2    50   Input ~ 0
+Currrent_ADC
 $EndSCHEMATC
