File: Hardware/stm32f103.sch (KiCad schematic (older format))
At the start: 13 parts, among them U2 STM32F103C8Tx

Commit message: Added LCSC part#, Thermal vias, etc
Parts:
- C4, C5, C6: LCSC (none) -> C28061
- C7: DigiKey (none) -> 732-8937-1-ND; LCSC (none) -> C43799
- C8: Lcsc (none) -> C28061
- C9: Digikey (none) -> 732-8851-1-ND; LCSC (none) -> C45671
- D1: LCSC (none) -> C193191
- R1, R2, R21, R22, R3: LCSC (none) -> C441891
- U2: LCSC (none) -> C8734
Changed lines of the file:
@@
 F 2 "Resistor_SMD:R_0603_1608Metric_Pad1.05x0.95mm_HandSolder" H 5400 1700 50  0001 C CNN
 F 3 "~" H 5400 1700 50  0001 C CNN
+F 4 "" V 5400 1700 50  0001 C CNN "Digikey"
+F 5 "C441891" V 5400 1700 50  0001 C CNN "LCSC"
 	1    5400 1700
 	0    1    1    0
@@
 F 2 "Resistor_SMD:R_0603_1608Metric_Pad1.05x0.95mm_HandSolder" H 4450 2200 50  0001 C CNN
 F 3 "~" H 4450 2200 50  0001 C CNN
+F 4 "" V 4450 2200 50  0001 C CNN "Digikey"
+F 5 "C441891" V 4450 2200 50  0001 C CNN "LCSC"
 	1    4450 2200
 	0    1    1    0
@@
 F 2 "Capacitor_SMD:C_0603_1608Metric_Pad1.05x0.95mm_HandSolder" H 8500 1750 50  0001 C CNN
 F 3 "~" H 8500 1750 50  0001 C CNN
+F 4 "" H 8500 1750 50  0001 C CNN "Digikey"
+F 5 "C28061" H 8500 1750 50  0001 C CNN "LCSC"
 	1    8500 1750
 	1    0    0    -1
@@
 F 2 "Capacitor_SMD:C_0603_1608Metric_Pad1.05x0.95mm_HandSolder" H 8900 1750 50  0001 C CNN
 F 3 "~" H 8900 1750 50  0001 C CNN
+F 4 "" H 8900 1750 50  0001 C CNN "Digikey"
+F 5 "C28061" H 8900 1750 50  0001 C CNN "LCSC"
 	1    8900 1750
 	1    0    0    -1
@@
 F 2 "Capacitor_SMD:C_0603_1608Metric_Pad1.05x0.95mm_HandSolder" H 9300 1750 50  0001 C CNN
 F 3 "~" H 9300 1750 50  0001 C CNN
+F 4 "" H 9300 1750 50  0001 C CNN "Digikey"
+F 5 "C28061" H 9300 1750 50  0001 C CNN "LCSC"
 	1    9300 1750
 	1    0    0    -1
@@
 F 2 "Capacitor_THT:CP_Radial_D5.0mm_P2.50mm" H 9700 1750 50  0001 C CNN
 F 3 "~" H 9700 1750 50  0001 C CNN
+F 4 "732-8937-1-ND" H 9700 1750 50  0001 C CNN "DigiKey"
+F 5 "C43799" H 9700 1750 50  0001 C CNN "LCSC"
 	1    9700 1750
 	1    0    0    -1
@@
 F 2 "Capacitor_SMD:C_0603_1608Metric_Pad1.05x0.95mm_HandSolder" H 10000 1750 50  0001 C CNN
 F 3 "~" H 10000 1750 50  0001 C CNN
+F 4 "" H 10000 1750 50  0001 C CNN "Digikey"
+F 5 "C28061" H 10000 1750 50  0001 C CNN "Lcsc"
 	1    10000 1750
 	1    0    0    -1
@@
 F 2 "Capacitor_THT:CP_Radial_D5.0mm_P2.50mm" H 10400 1750 50  0001 C CNN
 F 3 "~" H 10400 1750 50  0001 C CNN
+F 4 "732-8851-1-ND" H 10400 1750 50  0001 C CNN "Digikey"
+F 5 "C45671" H 10400 1750 50  0001 C CNN "LCSC"
 	1    10400 1750
 	1    0    0    -1
@@
 Wire Wire Line
 	5900 1800 6000 1800
-Wire Wire Line
-	6250 1600 6250 1800
-Wire Wire Line
-	6250 1800 6100 1800
 Text HLabel 4850 3600 0    50   Input ~ 0
 OLED_RST
@@
 L power:VDDA #PWR0122
 U 1 1 5F7D7644
-P 6250 1600
-F 0 "#PWR0122" H 6250 1450 50  0001 C CNN
-F 1 "VDDA" H 6265 1773 50  0000 C CNN
-F 2 "" H 6250 1600 50  0001 C CNN
-F 3 "" H 6250 1600 50  0001 C CNN
-	1    6250 1600
+P 6100 1600
+F 0 "#PWR0122" H 6100 1450 50  0001 C CNN
+F 1 "VDDA" H 6250 1775 50  0000 C CNN
+F 2 "" H 6100 1600 50  0001 C CNN
+F 3 "" H 6100 1600 50  0001 C CNN
+	1    6100 1600
 	1    0    0    -1
 $EndComp
@@
 F 2 "Capacitor_SMD:C_0805_2012Metric_Pad1.15x1.40mm_HandSolder" V 5050 5100 50  0001 C CNN
 F 3 "~" V 5050 5100 50  0001 C CNN
+F 4 "" V 5050 5100 50  0001 C CNN "Digikey"
+F 5 "C193191" V 5050 5100 50  0001 C CNN "LCSC"
 	1    5050 5100
 	0    -1   -1   0
@@
 F 2 "Resistor_SMD:R_0603_1608Metric_Pad1.05x0.95mm_HandSolder" H 5050 4775 50  0001 C CNN
 F 3 "~" H 5050 4775 50  0001 C CNN
+F 4 "" V 5050 4775 50  0001 C CNN "Digikey"
+F 5 "C441891" V 5050 4775 50  0001 C CNN "LCSC"
 	1    5050 4775
 	-1   0    0    1
@@
 F 2 "Package_QFP:LQFP-48_7x7mm_P0.5mm" H 5300 1900 50  0001 R CNN
 F 3 "http://www.st.com/st-web-ui/static/active/en/resource/technical/document/datasheet/CD00161566.pdf" H 5900 3300 50  0001 C CNN
+F 4 "" H 5900 3300 50  0001 C CNN "Digikey"
+F 5 "C8734" H 5900 3300 50  0001 C CNN "LCSC"
 	1    5900 3300
 	1    0    0    -1
@@
 F 2 "Resistor_SMD:R_0603_1608Metric_Pad1.05x0.95mm_HandSolder" H 4175 3325 50  0001 C CNN
 F 3 "~" H 4175 3325 50  0001 C CNN
+F 4 "" H 4175 3325 50  0001 C CNN "Digikey"
+F 5 "C441891" H 4175 3325 50  0001 C CNN "LCSC"
 	1    4175 3325
 	1    0    0    -1
@@
 F 2 "Resistor_SMD:R_0603_1608Metric_Pad1.05x0.95mm_HandSolder" H 4375 3300 50  0001 C CNN
 F 3 "~" H 4375 3300 50  0001 C CNN
+F 4 "" H 4375 3300 50  0001 C CNN "Digikey"
+F 5 "C441891" H 4375 3300 50  0001 C CNN "LCSC"
 	1    4375 3300
 	1    0    0    -1
@@
 Text HLabel 6850 3200 2    50   Input ~ 0
 Currrent_ADC
+Wire Wire Line
+	6100 1600 6100 1800
 $EndSCHEMATC

Commit message: Added second mosfet and added FPaste layer on thermal vias
Parts:
- C4, C5, C6: LCSC C28061 -> C1591
- C7: DigiKey 732-8937-1-ND -> (none); Digikey (none) -> 732-8937-1-ND
- C8: LCSC (none) -> C1591; Lcsc C28061 -> (none)
Changed lines of the file:
@@
 F 3 "~" H 8500 1750 50  0001 C CNN
 F 4 "" H 8500 1750 50  0001 C CNN "Digikey"
-F 5 "C28061" H 8500 1750 50  0001 C CNN "LCSC"
+F 5 "C1591" H 8500 1750 50  0001 C CNN "LCSC"
 	1    8500 1750
 	1    0    0    -1
@@
 F 3 "~" H 8900 1750 50  0001 C CNN
 F 4 "" H 8900 1750 50  0001 C CNN "Digikey"
-F 5 "C28061" H 8900 1750 50  0001 C CNN "LCSC"
+F 5 "C1591" H 8900 1750 50  0001 C CNN "LCSC"
 	1    8900 1750
 	1    0    0    -1
@@
 F 3 "~" H 9300 1750 50  0001 C CNN
 F 4 "" H 9300 1750 50  0001 C CNN "Digikey"
-F 5 "C28061" H 9300 1750 50  0001 C CNN "LCSC"
+F 5 "C1591" H 9300 1750 50  0001 C CNN "LCSC"
 	1    9300 1750
 	1    0    0    -1
@@
 F 2 "Capacitor_THT:CP_Radial_D5.0mm_P2.50mm" H 9700 1750 50  0001 C CNN
 F 3 "~" H 9700 1750 50  0001 C CNN
-F 4 "732-8937-1-ND" H 9700 1750 50  0001 C CNN "DigiKey"
+F 4 "732-8937-1-ND" H 9700 1750 50  0001 C CNN "Digikey"
 F 5 "C43799" H 9700 1750 50  0001 C CNN "LCSC"
 	1    9700 1750
@@
 F 3 "~" H 10000 1750 50  0001 C CNN
 F 4 "" H 10000 1750 50  0001 C CNN "Digikey"
-F 5 "C28061" H 10000 1750 50  0001 C CNN "Lcsc"
+F 5 "C1591" H 10000 1750 50  0001 C CNN "LCSC"
 	1    10000 1750
 	1    0    0    -1
