File: Hardware/Buttons.sch (KiCad schematic (older format))
At the start: 12 parts, among them SW2 SW_Push, SW3 SW_Push, SW4 SW_Push

Commit message: Added LCSC part#, Thermal vias, etc
Parts:
- C10: value 0.1uF -> 1u; LCSC (none) -> C696843
- C11, C12: LCSC (none) -> C696843
- R14, R15, R16, R17, R18, R19: LCSC (none) -> C441891
- SW2: Digikey (none) -> CKN9078-ND; LCSC (none) -> C221879
- SW3, SW4: LCSC (none) -> C221879
Changed lines of the file:
@@
 F 2 "Button_Switch_THT:SW_PUSH_6mm_H4.3mm" H 5000 3000 50  0001 C CNN
 F 3 "~" H 5000 3000 50  0001 C CNN
+F 4 "CKN9078-ND" H 5000 2800 50  0001 C CNN "Digikey"
+F 5 "C221879" H 5000 2800 50  0001 C CNN "LCSC"
 	1    5000 2800
 	1    0    0    -1
@@
 F 2 "Button_Switch_THT:SW_PUSH_6mm_H4.3mm" H 5000 3450 50  0001 C CNN
 F 3 "~" H 5000 3450 50  0001 C CNN
+F 4 "" H 5000 3250 50  0001 C CNN "Digikey"
+F 5 "C221879" H 5000 3250 50  0001 C CNN "LCSC"
 	1    5000 3250
 	1    0    0    -1
@@
 F 2 "Button_Switch_THT:SW_PUSH_6mm_H4.3mm" H 5000 3850 50  0001 C CNN
 F 3 "~" H 5000 3850 50  0001 C CNN
+F 4 "" H 5000 3650 50  0001 C CNN "Digikey"
+F 5 "C221879" H 5000 3650 50  0001 C CNN "LCSC"
 	1    5000 3650
 	1    0    0    -1
@@
 F 2 "Resistor_SMD:R_0603_1608Metric_Pad1.05x0.95mm_HandSolder" H 6600 2800 50  0001 C CNN
 F 3 "~" H 6600 2800 50  0001 C CNN
+F 4 "" V 6600 2800 50  0001 C CNN "Digikey"
+F 5 "C441891" V 6600 2800 50  0001 C CNN "LCSC"
 	1    6600 2800
 	0    1    1    0
@@
 F 2 "Resistor_SMD:R_0603_1608Metric_Pad1.05x0.95mm_HandSolder" H 6575 3250 50  0001 C CNN
 F 3 "~" H 6575 3250 50  0001 C CNN
+F 4 "" V 6575 3250 50  0001 C CNN "Digikey"
+F 5 "C441891" V 6575 3250 50  0001 C CNN "LCSC"
 	1    6575 3250
 	0    1    1    0
@@
 F 2 "Resistor_SMD:R_0603_1608Metric_Pad1.05x0.95mm_HandSolder" H 6575 3650 50  0001 C CNN
 F 3 "~" H 6575 3650 50  0001 C CNN
+F 4 "" V 6575 3650 50  0001 C CNN "Digikey"
+F 5 "C441891" V 6575 3650 50  0001 C CNN "LCSC"
 	1    6575 3650
 	0    1    1    0
@@
 P 6750 2900
 F 0 "C10" H 6842 2946 50  0000 L CNN
-F 1 "0.1uF" H 6842 2855 50  0000 L CNN
+F 1 "1u" H 6842 2855 50  0000 L CNN
 F 2 "Capacitor_SMD:C_0603_1608Metric_Pad1.05x0.95mm_HandSolder" H 6750 2900 50  0001 C CNN
 F 3 "~" H 6750 2900 50  0001 C CNN
+F 4 "" H 6750 2900 50  0001 C CNN "Digikey"
+F 5 "C696843" H 6750 2900 50  0001 C CNN "LCSC"
 	1    6750 2900
 	1    0    0    -1
@@
 F 2 "Capacitor_SMD:C_0603_1608Metric_Pad1.05x0.95mm_HandSolder" H 6725 3350 50  0001 C CNN
 F 3 "~" H 6725 3350 50  0001 C CNN
+F 4 "" H 6725 3350 50  0001 C CNN "Digikey"
+F 5 "C696843" H 6725 3350 50  0001 C CNN "LCSC"
 	1    6725 3350
 	1    0    0    -1
@@
 F 2 "Capacitor_SMD:C_0603_1608Metric_Pad1.05x0.95mm_HandSolder" H 6725 3750 50  0001 C CNN
 F 3 "~" H 6725 3750 50  0001 C CNN
+F 4 "" H 6725 3750 50  0001 C CNN "Digikey"
+F 5 "C696843" H 6725 3750 50  0001 C CNN "LCSC"
 	1    6725 3750
 	1    0    0    -1
@@
 F 2 "Resistor_SMD:R_0603_1608Metric_Pad1.05x0.95mm_HandSolder" H 5950 2600 50  0001 C CNN
 F 3 "~" H 5950 2600 50  0001 C CNN
+F 4 "" H 5950 2600 50  0001 C CNN "Digikey"
+F 5 "C441891" H 5950 2600 50  0001 C CNN "LCSC"
 	1    5950 2600
 	-1   0    0    1
@@
 F 2 "Resistor_SMD:R_0603_1608Metric_Pad1.05x0.95mm_HandSolder" H 6150 3050 50  0001 C CNN
 F 3 "~" H 6150 3050 50  0001 C CNN
+F 4 "" H 6150 3050 50  0001 C CNN "Digikey"
+F 5 "C441891" H 6150 3050 50  0001 C CNN "LCSC"
 	1    6150 3050
 	-1   0    0    1
@@
 F 2 "Resistor_SMD:R_0603_1608Metric_Pad1.05x0.95mm_HandSolder" H 6400 3450 50  0001 C CNN
 F 3 "~" H 6400 3450 50  0001 C CNN
+F 4 "" H 6400 3450 50  0001 C CNN "Digikey"
+F 5 "C441891" H 6400 3450 50  0001 C CNN "LCSC"
 	1    6400 3450
 	-1   0    0    1

Commit message: Added second mosfet and added FPaste layer on thermal vias
Parts:
- C10: value 1u -> 1uF
- R14, R15, R16, R17, R18, R19: value 1K -> 1k
Changed lines of the file:
@@
 P 6600 2800
 F 0 "R14" V 6404 2800 50  0000 C CNN
-F 1 "1K" V 6495 2800 50  0000 C CNN
+F 1 "1k" V 6495 2800 50  0000 C CNN
 F 2 "Resistor_SMD:R_0603_1608Metric_Pad1.05x0.95mm_HandSolder" H 6600 2800 50  0001 C CNN
 F 3 "~" H 6600 2800 50  0001 C CNN
@@
 P 6575 3250
 F 0 "R15" V 6379 3250 50  0000 C CNN
-F 1 "1K" V 6470 3250 50  0000 C CNN
+F 1 "1k" V 6470 3250 50  0000 C CNN
 F 2 "Resistor_SMD:R_0603_1608Metric_Pad1.05x0.95mm_HandSolder" H 6575 3250 50  0001 C CNN
 F 3 "~" H 6575 3250 50  0001 C CNN
@@
 P 6575 3650
 F 0 "R16" V 6379 3650 50  0000 C CNN
-F 1 "1K" V 6470 3650 50  0000 C CNN
+F 1 "1k" V 6470 3650 50  0000 C CNN
 F 2 "Resistor_SMD:R_0603_1608Metric_Pad1.05x0.95mm_HandSolder" H 6575 3650 50  0001 C CNN
 F 3 "~" H 6575 3650 50  0001 C CNN
@@
 P 6750 2900
 F 0 "C10" H 6842 2946 50  0000 L CNN
-F 1 "1u" H 6842 2855 50  0000 L CNN
+F 1 "1uF" H 6842 2855 50  0000 L CNN
 F 2 "Capacitor_SMD:C_0603_1608Metric_Pad1.05x0.95mm_HandSolder" H 6750 2900 50  0001 C CNN
 F 3 "~" H 6750 2900 50  0001 C CNN
@@
 P 5950 2600
 F 0 "R17" H 5891 2554 50  0000 R CNN
-F 1 "1K" H 5891 2645 50  0000 R CNN
+F 1 "1k" H 5891 2645 50  0000 R CNN
 F 2 "Resistor_SMD:R_0603_1608Metric_Pad1.05x0.95mm_HandSolder" H 5950 2600 50  0001 C CNN
 F 3 "~" H 5950 2600 50  0001 C CNN
@@
 P 6150 3050
 F 0 "R18" H 6091 3004 50  0000 R CNN
-F 1 "1K" H 6091 3095 50  0000 R CNN
+F 1 "1k" H 6091 3095 50  0000 R CNN
 F 2 "Resistor_SMD:R_0603_1608Metric_Pad1.05x0.95mm_HandSolder" H 6150 3050 50  0001 C CNN
 F 3 "~" H 6150 3050 50  0001 C CNN
@@
 P 6400 3450
 F 0 "R19" H 6600 3425 50  0000 R CNN
-F 1 "1K" H 6575 3525 50  0000 R CNN
+F 1 "1k" H 6575 3525 50  0000 R CNN
 F 2 "Resistor_SMD:R_0603_1608Metric_Pad1.05x0.95mm_HandSolder" H 6400 3450 50  0001 C CNN
 F 3 "~" H 6400 3450 50  0001 C CNN
